File: PCB_.kicad_pcb (KiCad board)
At the start: 2 copper layers, 58 x 34 mm, 24 parts, among them J1 ST7735, J2 DS18B20, J3 TL494, J4 INA226, J5 FAN_CTRL, J6 PWR, J7 SWD, SW1 RST, U1 STM32F030F4P6, U2 AMS1117-3.3, Y1 Crystal

Commit message: start tracing
Parts:
- added R3: 0R, Resistor_SMD:R_1206_3216Metric_Pad1.30x1.75mm_HandSolder, F.Cu at (153.9, 68.2)
- added R5: 0R, Resistor_SMD:R_1206_3216Metric_Pad1.30x1.75mm_HandSolder, F.Cu at (153.9, 70.8)
- added R6: 0R, Resistor_SMD:R_1206_3216Metric_Pad1.30x1.75mm_HandSolder, F.Cu at (153.9, 73.5)
- added R7: 100R, Resistor_SMD:R_1206_3216Metric_Pad1.30x1.75mm_HandSolder, F.Cu at (153.9, 77.0)
- J7: footprint Connector_PinHeader_2.54mm:PinHeader_1x03_P2.54mm_Vertical -> Connector_PinHeader_2.54mm:PinHeader_1x04_P2.54mm_Vertical
- moved J1 17.8 mm to (148.2, 62.8), turned to 180 degrees
- moved R2 11.8 mm to (168.8, 64.0)
- moved J3 8.06 mm to (152.5, 60.5)
- moved R4 6.34 mm to (168.8, 66.8)
- moved J7 6.33 mm to (169.7, 78.2), turned to -90 degrees
- moved J4 6.00 mm to (168.5, 85.5)
- moved SW1 4.34 mm to (176.8, 67.2)
- moved C6 3.82 mm to (181.2, 57.8)
- moved C7 3.55 mm to (149.8, 56.5)
- moved C5 2.85 mm to (168.8, 72.0)
- moved R1 2.50 mm to (168.8, 69.5)
- moved J5 1.58 mm to (153.0, 81.0)
- moved C4 1.57 mm to (161.5, 64.7)
- moved U1 1.24 mm to (161.6, 71.6)
- moved C2 0.79 mm to (161.8, 78.5)
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Connections:
- J1 pad 4: DISP_DC -> Net-(J1-Pin_4)
- J1 pad 5: DISP_RST -> Net-(J1-Pin_5)
- J1 pad 6: DISP_CS -> Net-(J1-Pin_6)
- J5 pad 1: FAN_PWM -> Net-(J5-Pin_1)
Routing:
- net DISP_SDA: track 0.00 -> 26.9 mm
- net DISP_SCK: track 0.00 -> 20.9 mm
- net DISP_DC: track 0.00 -> 7.61 mm
- net FAN_PWM: track 0.00 -> 5.41 mm
- net Net-(J1-Pin_4): track 0.00 -> 5.32 mm
- net Net-(J1-Pin_6): track 0.00 -> 5.25 mm
- net Net-(J1-Pin_5): track 0.00 -> 5.19 mm
- net DISP_RST: track 0.00 -> 5.18 mm
- net Net-(J5-Pin_1): track 0.00 -> 4.25 mm
- net DISP_CS: track 0.00 -> 3.34 mm

Commit message: MCU tracing is done
Parts:
- added R8: 5.1K, Resistor_SMD:R_0805_2012Metric_Pad1.20x1.40mm_HandSolder, F.Cu at (152.0, 84.2)
- J7: footprint Connector_PinHeader_2.54mm:PinHeader_1x04_P2.54mm_Vertical -> Connector_PinHeader_2.54mm:PinHeader_1x05_P2.54mm_Vertical
- moved C9 28.5 mm to (176.2, 84.5), turned to -90 degrees
- moved U2 18.4 mm to (182.5, 83.2), turned to 180 degrees
- moved J6 7.29 mm to (188.5, 73.8)
- moved C8 6.54 mm to (187.0, 77.5)
- moved J4 4.86 mm to (169.5, 80.8)
- moved R2 3.50 mm to (165.2, 64.0)
- moved C6 3.25 mm to (178.0, 57.8)
- moved J2 3.01 mm to (161.2, 84.5)
- moved C7 2.57 mm to (152.0, 57.8)
- moved J7 2.50 mm to (168.2, 76.2)
- moved SW1 2.12 mm to (177.5, 69.2), turned to -90 degrees
- moved C4 1.42 mm to (160.5, 63.8), turned to 180 degrees
- moved J5 0.90 mm to (152.2, 80.5)
- moved C5 0.88 mm to (169.2, 72.8)
- moved J3 0.75 mm to (152.5, 61.2)
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Connections:
- J2 pad 2: TEMP -> GND
- J2 pad 3: GND -> TEMP
- J7 pad 1: +3V3 -> SWCLK
- J7 pad 3: SWCLK -> SW_RST
Routing:
- net +3V3: track 0.00 -> 105.7 mm
- net SW_RST: track 0.00 -> 37.3 mm
- net GND: track 0.00 -> 36.9 mm, vias 0 -> 10
- net OSC_OUT: track 0.00 -> 22.0 mm
- net OSC_IN: track 0.00 -> 21.3 mm
- net TEMP: track 0.00 -> 16.3 mm
- net DISP_LED: track 0.00 -> 15.9 mm
- net 494_ON: track 0.00 -> 14.0 mm
- net I2C_SDA: track 0.00 -> 11.0 mm
- net SWDIO: track 0.00 -> 10.6 mm
- net +5V: track 0.00 -> 9.43 mm
- net I2C_SCL: track 0.00 -> 9.43 mm
- net Net-(U1-VDDA): track 0.00 -> 7.46 mm
- net SWCLK: track 0.00 -> 4.50 mm
- net Net-(U1-BOOT0): track 0.00 -> 3.02 mm
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- added copper zone on B.Cu, net GND
